Commit message: Improve obstacle support + urdf generation - urdfs are now autogenerated - full maps can be used directly by the planner

File: maps/landing.urdf (robot description, URDF)
Before this commit: robot wall_a.urdf, 1 links, 0 joints
Links:
- link baseLink: geometry collision box size=0.3 0.3 0.3; visual mesh filename=cube.obj scale=0.3 0.3 0.3

File: maps/take_off.urdf (robot description, URDF)
Before this commit: robot wall_a.urdf, 1 links, 0 joints
Links:
- link baseLink: geometry collision box size=0.3 0.3 0.3; visual mesh filename=cube.obj scale=0.3 0.3 0.3
