Commit message: merge input and profiling further

File: maps/obstacles/wall_a.urdf (robot description, URDF)
Before this commit: robot wall_a.urdf, 1 links, 0 joints
Links:
- link baseLink: geometry collision box size=1.5 0.1 0.6; visual mesh filename=cube.obj scale=1.5 0.1 0.6

File: maps/obstacles/wall_b.urdf (robot description, URDF)
Before this commit: robot wall_b.urdf, 1 links, 0 joints
Links:
- link baseLink: geometry collision box size=2 0.1 1.2; visual mesh filename=cube.obj scale=2 0.1 1.2

File: maps/obstacles/wall_c.urdf (robot description, URDF)
Before this commit: robot wall_c.urdf, 1 links, 0 joints
Links:
- link baseLink: geometry collision box size=1.4 0.1 1.2; visual mesh filename=cube.obj scale=1.4 0.1 1.2

File: maps/obstacles/wall_d.urdf (robot description, URDF)
Before this commit: robot wall_d.urdf, 1 links, 0 joints
Links:
- link baseLink: geometry collision box size=0.1 1.15 1.2; visual mesh filename=cube.obj scale=0.1 1.15 1.2
